Commit message: updated URDF supporting relative filepaths

File: A-2240-06G.urdf (robot description, URDF)
Before this commit: robot A-2240-06G, 26 links, 25 joints
Links:
- link J1/body: geometry collision mesh filename=hebi_description/meshes/R8.stl scale=0.001 0.001 0.001; visual mesh filename=hebi_description/meshes/R8.stl scale=0.001 0.001 0.001
- link J2/body: geometry collision mesh filename=hebi_description/meshes/R8.stl scale=0.001 0.001 0.001; visual mesh filename=hebi_description/meshes/R8.stl scale=0.001 0.001 0.001
- link J3/body: geometry collision mesh filename=hebi_description/meshes/R8.stl scale=0.001 0.001 0.001; visual mesh filename=hebi_description/meshes/R8.stl scale=0.001 0.001 0.001
- link J4/body: geometry collision mesh filename=hebi_description/meshes/R8.stl scale=0.001 0.001 0.001; visual mesh filename=hebi_description/meshes/R8.stl scale=0.001 0.001 0.001
- link J5/body: geometry collision mesh filename=hebi_description/meshes/R8.stl scale=0.001 0.001 0.001; visual mesh filename=hebi_description/meshes/R8.stl scale=0.001 0.001 0.001
- link J6/body: geometry collision mesh filename=hebi_description/meshes/R8.stl scale=0.001 0.001 0.001; visual mesh filename=hebi_description/meshes/R8.stl scale=0.001 0.001 0.001
- link bracket_1: geometry collision mesh filename=hebi_description/meshes/A-2221-01-Outside.stl scale=0.001 0.001 0.001; visual mesh filename=hebi_description/meshes/A-2221-01-Outside.stl scale=0.001 0.001 0.001
- link bracket_2: geometry collision mesh filename=hebi_description/meshes/A-2220-01.stl scale=0.001 0.001 0.001; visual mesh filename=hebi_description/meshes/A-2220-01.stl scale=0.001 0.001 0.001
- link bracket_3: geometry collision mesh filename=hebi_description/meshes/A-2220-01.stl scale=0.001 0.001 0.001; visual mesh filename=hebi_description/meshes/A-2220-01.stl scale=0.001 0.001 0.001
- link end_effector_1/center_hub: geometry collision mesh filename=hebi_description/meshes/PM-2357-02.stl scale=0.001 0.001 0.001; visual mesh filename=hebi_description/meshes/PM-2357-02.stl scale=0.001 0.001 0.001
- link end_effector_1/center_pinion: geometry collision mesh filename=hebi_description/meshes/PM-2291-01.stl scale=0.001 0.001 0.001; visual mesh filename=hebi_description/meshes/PM-2291-01.stl scale=0.001 0.001 0.001
- link end_effector_1/l_finger: geometry collision mesh filename=hebi_description/meshes/PM-2221-01.stl scale=0.001 0.001 0.001; visual mesh filename=hebi_description/meshes/PM-2221-01.stl scale=0.001 0.001 0.001
- link end_effector_1/l_gripper: geometry collision mesh filename=hebi_description/meshes/PM-2360-02.stl scale=0.001 0.001 0.001; visual mesh filename=hebi_description/meshes/PM-2360-02.stl scale=0.001 0.001 0.001
- link end_effector_1/l_inner_linkage: geometry collision mesh filename=hebi_description/meshes/PM-2359-02.stl scale=0.001 0.001 0.001; visual mesh filename=hebi_description/meshes/PM-2359-02.stl scale=0.001 0.001 0.001
- link end_effector_1/l_outer_linkage: geometry collision mesh filename=hebi_description/meshes/PM-2358-02.stl scale=0.001 0.001 0.001; visual mesh filename=hebi_description/meshes/PM-2358-02.stl scale=0.001 0.001 0.001
- link end_effector_1/r_finger: geometry collision mesh filename=hebi_description/meshes/PM-2221-01.stl scale=0.001 0.001 0.001; visual mesh filename=hebi_description/meshes/PM-2221-01.stl scale=0.001 0.001 0.001
- link end_effector_1/r_gripper: geometry collision mesh filename=hebi_description/meshes/PM-2360-02.stl scale=0.001 0.001 0.001; visual mesh filename=hebi_description/meshes/PM-2360-02.stl scale=0.001 0.001 0.001
- link end_effector_1/r_inner_linkage: geometry collision mesh filename=hebi_description/meshes/PM-2359-02.stl scale=0.001 0.001 0.001; visual mesh filename=hebi_description/meshes/PM-2359-02.stl scale=0.001 0.001 0.001
- link end_effector_1/r_outer_linkage: geometry collision mesh filename=hebi_description/meshes/PM-2358-02.stl scale=0.001 0.001 0.001; visual mesh filename=hebi_description/meshes/PM-2358-02.stl scale=0.001 0.001 0.001
- link link_1: geometry collision cylinder length=0.29960000000000003 radius=.016; collision mesh filename=hebi_description/meshes/A-2038-02.stl scale=0.001 0.001 0.001
- link link_2: geometry collision cylinder length=0.29960000000000003 radius=.016; collision mesh filename=hebi_description/meshes/A-2038-02.stl scale=0.001 0.001 0.001
