Commit message: working joint-only BC pipeline: loss curves + hyperparameter sweep, pre-vision

File: A-2240-06G.urdf (robot description, URDF)
Before this commit: robot A-2240-06G, 26 links, 25 joints
Links:
- link J1/body: geometry collision mesh filename=hebi_description/meshes/R8.stl scale=0.001 0.001 0.001
- link J2/body: geometry collision mesh filename=hebi_description/meshes/R8.stl scale=0.001 0.001 0.001
- link J3/body: geometry collision mesh filename=hebi_description/meshes/R8.stl scale=0.001 0.001 0.001
- link J4/body: geometry collision mesh filename=hebi_description/meshes/R8.stl scale=0.001 0.001 0.001
- link J5/body: geometry collision mesh filename=hebi_description/meshes/R8.stl scale=0.001 0.001 0.001
- link J6/body: geometry collision mesh filename=hebi_description/meshes/R8.stl scale=0.001 0.001 0.001
- link bracket_1: geometry collision mesh filename=hebi_description/meshes/A-2221-01-Outside.stl scale=0.001 0.001 0.001
- link bracket_3: geometry collision mesh filename=hebi_description/meshes/A-2220-01.stl scale=0.001 0.001 0.001
- link end_effector_1/l_inner_linkage: geometry collision box size=0.01 0.005 0.04
- link end_effector_1/r_inner_linkage: geometry collision box size=0.01 0.005 0.04
- link link_1: geometry collision cylinder length=0.29960000000000003 radius=.016; collision mesh filename=hebi_description/meshes/A-2038-02.stl scale=0.001 0.001 0.001
- link link_2: geometry collision cylinder length=0.29960000000000003 radius=.016; collision mesh filename=hebi_description/meshes/A-2038-02.stl scale=0.001 0.001 0.001
